Commit message: add customized bumper2pc (point cloud); use estimated_pose instead of mapping specific amcl_pose; do not launch fake_ocalization for two turtlebots (manually launch localization from chris_turtlebot_navigation instead)

File: chris_turtlebot_model/urdf/kobuki_gazebo.urdf.xacro (robot description, xacro)
@@ -36,6 +36,6 @@
     </gazebo>
     <gazebo reference="base_link">
-      <mu1>0.3</mu1>
-      <mu2>0.3</mu2>
+      <mu1>10</mu1>
+      <mu2>10</mu2>
       <sensor type="contact" name="bumpers">
         <always_on>1</always_on>
@@ -43,5 +43,5 @@
         <visualize>true</visualize>
         <contact>
-          <collision>base_footprint_collision_base_link</collision>
+          <collision>base_footprint_fixed_joint_lump__base_link_collision</collision>
         </contact>
       </sensor>
