Commit message: Begin integration of EGOKITUZ Kobuki Turtlebot

File: chris_turtlebot_model/robots/chris_turtlebot.urdf.xacro (robot description, xacro)
@@ -4,16 +4,10 @@
   <xacro:include filename="$(find turtlebot_description)/urdf/turtlebot_common_library.urdf.xacro" />
   <xacro:include filename="$(find chris_turtlebot_model)/urdf/kobuki.urdf.xacro" />
-  <xacro:include filename="$(find turtlebot_description)/urdf/stacks/hexagons.urdf.xacro"/>
-  <xacro:include filename="$(find turtlebot_description)/urdf/sensors/kinect.urdf.xacro"/>
-  <xacro:include filename="$(find chris_turtlebot_model)/urdf/hokuyo_urg04.urdf.xacro"/>
-  <kobuki/>
-  <stack_hexagons parent="base_footprint"/>
-  <sensor_kinect  parent="base_footprint"/>
-  <joint name="hokuyo_base_joint" type="fixed">
-    <axis xyz="0 0 1" />
-    <origin xyz="-0.0254 0.0 0.208" rpy="0 0 0"/>
-    <parent link="base_footprint"/>
-    <child link="hokuyo_base_link"/>
-  </joint>
-  <xacro:hokuyo_urg04 lidar_name="hokuyo"/>
+  <xacro:include filename="$(find turtlebot_description)/urdf/stacks/egokituz.urdf.xacro"/>
+  <xacro:include filename="$(find turtlebot_description)/urdf/sensors/d435.urdf.xacro"/>
+  <xacro:include filename="$(find turtlebot_description)/urdf/sensors/ydlidar_x4.urdf.xacro"/>
+  <xacro:kobuki/>
+  <xacro:stack_hexagons parent="base_link"/>
+  <xacro:sensor_d435    parent="base_link"/>
+  <xacro:ydlidar_x4 name="ydlidar" base="base_link" pose_xyz="0.0195 -0.005 0.225" pose_rpy="0 0 ${-1*M_PI}" />
 </robot>
